File: schematic_electrical/PROX_SENSE_LEVEL_SHIFT.kicad_sch (KiCad schematic)
At the start: 8 parts, among them U2 HILETGO_LEVEL_SHIFT_1V8_6V0, U3 HILETGO_LEVEL_SHIFT_1V8_6V0, U5 ULN2803A

Commit message: Pylon schmatic: clarify filenames and add orange text to avoid confusing other similar schematic pages.
Other:
- note added: "PYLONS"
Changed lines of the file:
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@@
+		)
+	)
+	(text "PYLONS"
+		(exclude_from_sim no)
+		(at 29.718 22.098 0)
+		(effects
+			(font
+				(size 4.7752 4.7752)
+				(thickness 0.955)
+				(bold yes)
+				(italic yes)
+				(color 255 153 0 1)
+			)
 		)
 	)
@@
 		)
 		(instances
-			(project "high_striker_boosh"
+			(project "pylons_boosh_remote_reciver"
 				(path "/f3653ac0-a28a-4ee8-bcf5-236139001455/a54607f4-b6e0-4e44-9873-c16ace68b07d"
 					(reference "U2")
@@
 		)
 		(instances
-			(project "high_striker_boosh"
+			(project "pylons_boosh_remote_reciver"
 				(path "/f3653ac0-a28a-4ee8-bcf5-236139001455/a54607f4-b6e0-4e44-9873-c16ace68b07d"
 					(reference "R16")
@@
 		)
 		(instances
-			(project "high_striker_boosh"
+			(project "pylons_boosh_remote_reciver"
 				(path "/f3653ac0-a28a-4ee8-bcf5-236139001455/a54607f4-b6e0-4e44-9873-c16ace68b07d"
 					(reference "#PWR011")
@@
 		)
 		(instances
-			(project "high_striker_boosh"
+			(project "pylons_boosh_remote_reciver"
 				(path "/f3653ac0-a28a-4ee8-bcf5-236139001455/a54607f4-b6e0-4e44-9873-c16ace68b07d"
 					(reference "#PWR06")
@@
 		)
 		(instances
-			(project "high_striker_boosh"
+			(project "pylons_boosh_remote_reciver"
 				(path "/f3653ac0-a28a-4ee8-bcf5-236139001455/a54607f4-b6e0-4e44-9873-c16ace68b07d"
 					(reference "R15")
@@
 		)
 		(instances
-			(project "high_striker_boosh"
+			(project "pylons_boosh_remote_reciver"
 				(path "/f3653ac0-a28a-4ee8-bcf5-236139001455/a54607f4-b6e0-4e44-9873-c16ace68b07d"
 					(reference "R14")
@@
 		)
 		(instances
-			(project "high_striker_boosh"
+			(project "pylons_boosh_remote_reciver"
 				(path "/f3653ac0-a28a-4ee8-bcf5-236139001455/a54607f4-b6e0-4e44-9873-c16ace68b07d"
 					(reference "U5")
@@
 		)
 		(instances
-			(project "high_striker_boosh"
+			(project "pylons_boosh_remote_reciver"
 				(path "/f3653ac0-a28a-4ee8-bcf5-236139001455/a54607f4-b6e0-4e44-9873-c16ace68b07d"
 					(reference "R4")
@@
 		)
 		(instances
-			(project "high_striker_boosh"
+			(project "pylons_boosh_remote_reciver"
 				(path "/f3653ac0-a28a-4ee8-bcf5-236139001455/a54607f4-b6e0-4e44-9873-c16ace68b07d"
 					(reference "#PWR050")
@@
 		)
 		(instances
-			(project "high_striker_boosh"
+			(project "pylons_boosh_remote_reciver"
 				(path "/f3653ac0-a28a-4ee8-bcf5-236139001455/a54607f4-b6e0-4e44-9873-c16ace68b07d"
 					(reference "U3")
@@
 		)
 		(instances
-			(project "high_striker_boosh"
+			(project "pylons_boosh_remote_reciver"
 				(path "/f3653ac0-a28a-4ee8-bcf5-236139001455/a54607f4-b6e0-4e44-9873-c16ace68b07d"
 					(reference "#PWR09")
@@
 		)
 		(instances
-			(project "high_striker_boosh"
+			(project "pylons_boosh_remote_reciver"
 				(path "/f3653ac0-a28a-4ee8-bcf5-236139001455/a54607f4-b6e0-4e44-9873-c16ace68b07d"
 					(reference "R5")
@@
 		)
 		(instances
-			(project "high_striker_boosh"
+			(project "pylons_boosh_remote_reciver"
 				(path "/f3653ac0-a28a-4ee8-bcf5-236139001455/a54607f4-b6e0-4e44-9873-c16ace68b07d"
 					(reference "#PWR08")
@@
 		)
 		(instances
-			(project "high_striker_boosh"
+			(project "pylons_boosh_remote_reciver"
 				(path "/f3653ac0-a28a-4ee8-bcf5-236139001455/a54607f4-b6e0-4e44-9873-c16ace68b07d"
 					(reference "#PWR05")
@@
 		)
 		(instances
-			(project "high_striker_boosh"
+			(project "pylons_boosh_remote_reciver"
 				(path "/f3653ac0-a28a-4ee8-bcf5-236139001455/a54607f4-b6e0-4e44-9873-c16ace68b07d"
 					(reference "#PWR048")
@@
 		)
 		(instances
-			(project "high_striker_boosh"
+			(project "pylons_boosh_remote_reciver"
 				(path "/f3653ac0-a28a-4ee8-bcf5-236139001455/a54607f4-b6e0-4e44-9873-c16ace68b07d"
 					(reference "#PWR010")
