File: schematic_electrical/BOOSH_TRIGGER.kicad_sch (KiCad schematic)
At the start: 15 parts, among them Q1 FQP27P06, Q2 FQP27P06, U4 ULN2803A

Commit message: Add expansion buttons/lamps schematic sheet; schematic cleanup and annotations
- New EXPANSION_BUTTONS_LAMPS.kicad_sch sheet wired into top-level schematic
- Add AB_800T-QT24 symbol library
- ESP32_MCU: wire previously unconnected GPIO pins to BUTTON0-4 and BUTTON_LAMP_PWM_OUT0-4 global labels; add expansion IO bounding box annotation
- POWER: add GND ganging fabrication notes, DCDC USB wiring note, fuse value updated to "10A MINI AUTO BLADE"; routing cleanup
- CONNECTORS: routing and junction cleanup
- BOOSH_TRIGGER: remove stale "1R" errata note
- IDEA.md: add sandbox notes and open questions

Co-Authored-By: Claude Sonnet 4.6 <noreply@anthropic.com>
Other:
- note removed: "ONE BOARD MISTAKENLY USES 1R HERE!"
Changed lines of the file:
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@@
-		)
-	)
-	(text "ONE BOARD MISTAKENLY \nUSES 1R HERE!"
-		(exclude_from_sim no)
-		(at 215.9 54.864 0)
-		(effects
-			(font
-				(size 1.27 1.27)
-			)
 		)
 	)
