File: schematic_electrical/CONNECTORS.kicad_sch (KiCad schematic)
At the start: 10 parts, among them J1 Conn_01x02, J12 Conn_01x03, J15 Conn_01x02, J16 Conn_01x03, J2 Conn_01x02, J3 2-pin red PCB mount connector, J4 2-pin red PCB mount connector, J5 2-pin red PCB mount connector

Commit message: Recalibrate thermistor, add reset reason to web UI, increase LED brightness
- Thermistor 2-point calibration redone with equilibrated reference points
  (48.3°F and 116°F); prior calibration used a non-equilibrated 156.9°F point
  that produced a bad slope. New: scale=0.9116, offset=+13.92°F
- Add last_reset_reason to telemetry API and web UI (esp_reset_reason())
- Increase PWM LED brightness from 33% to 66% duty cycle
- Schematic: update R8 value label to 22k (as built), clean CONNECTORS page

Co-Authored-By: Claude Sonnet 4.6 <noreply@anthropic.com>
Parts:
- removed J4: 2-pin red PCB mount connector, symbol Connector_Generic:Conn_01x02
Other:
- note added: "YELLOW 16-GA FLYWIRE"
Changed lines of the file:
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@@
-	)
-	(junction
-		(at 191.77 35.56)
-		(diameter 0)
-		(color 0 0 0 0)
 	)
 	(junction
@@
 	)
 	(junction
-		(at 179.07 33.02)
-		(diameter 0)
-		(color 0 0 0 0)
-	)
-	(junction
-		(at 167.64 64.77)
-		(diameter 0)
-		(color 0 0 0 0)
-	)
-	(junction
 		(at 132.08 67.31)
 		(diameter 0)
@@
 	(wire
 		(pts
-			(xy 191.77 35.56) (xy 191.77 38.1)
-		)
-		(stroke
-			(width 0.508)
-			(type default)
-		)
-	)
-	(wire
-		(pts
 			(xy 138.43 44.45) (xy 134.62 44.45)
 		)
@@
 	(wire
 		(pts
-			(xy 167.64 35.56) (xy 191.77 35.56)
-		)
-		(stroke
-			(width 0.508)
-			(type default)
-		)
-	)
-	(wire
-		(pts
 			(xy 279.4 64.77) (xy 248.92 64.77)
 		)
@@
 	(wire
 		(pts
-			(xy 179.07 33.02) (xy 191.77 33.02)
-		)
-		(stroke
-			(width 0.508)
-			(type default)
-		)
-	)
-	(wire
-		(pts
 			(xy 130.81 129.54) (xy 100.33 129.54)
 		)
@@
 	(wire
 		(pts
-			(xy 142.24 64.77) (xy 167.64 64.77)
+			(xy 142.24 64.77) (xy 205.74 64.77)
 		)
 		(stroke
@@
 	(wire
 		(pts
-			(xy 167.64 64.77) (xy 205.74 64.77)
-		)
-		(stroke
-			(width 0.508)
-			(type default)
-		)
-	)
-	(wire
-		(pts
 			(xy 134.62 44.45) (xy 130.81 44.45)
 		)
@@
 		(pts
 			(xy 275.59 59.69) (xy 275.59 92.71)
-		)
-		(stroke
-			(width 0.508)
-			(type default)
-		)
-	)
-	(wire
-		(pts
-			(xy 167.64 35.56) (xy 167.64 64.77)
 		)
 		(stroke
@@
 			(font
 				(size 1.524 1.524)
+			)
+		)
+	)
+	(text "YELLOW 16-GA FLYWIRE"
+		(exclude_from_sim no)
+		(at 191.262 32.766 0)
+		(effects
+			(font
+				(size 1.27 1.27)
 			)
 		)
@@
 				(justify right)
 				(hide yes)
-			)
-		)
-	)
-	(symbol
-		(lib_id "Connector_Generic:Conn_01x02")
-		(at 196.85 33.02 0)
-		(unit 1)
-		(exclude_from_sim no)
-		(in_bom yes)
-		(on_board yes)
-		(dnp no)
-		(property "Reference" "J4"
-			(at 199.39 33.0199 0)
-			(effects
-				(font
-					(size 1.27 1.27)
-				)
-				(justify left)
-			)
-		)
-		(property "Value" "2-pin red PCB mount connector"
-			(at 199.39 35.5599 0)
-			(effects
-				(font
-					(size 1.27 1.27)
-				)
-				(justify left)
-			)
-		)
-		(property "Footprint" ""
-			(at 196.85 33.02 0)
-			(effects
-				(font
-					(size 1.27 1.27)
-				)
-				(hide yes)
-			)
-		)
-		(property "Datasheet" "~"
-			(at 196.85 33.02 0)
-			(effects
-				(font
-					(size 1.27 1.27)
-				)
-				(hide yes)
-			)
-		)
-		(property "Description" "Generic connector, single row, 01x02, script generated (kicad-library-utils/schlib/autogen/connector/)"
-			(at 196.85 33.02 0)
-			(effects
-				(font
-					(size 1.27 1.27)
-				)
-				(hide yes)
-			)
-		)
-		(pin "2"
-		)
-		(pin "1"
-		)
-		(instances
-			(project "pylons_boosh_remote_reciver"
-				(path "/f3653ac0-a28a-4ee8-bcf5-236139001455/d08cb7b6-6190-46a9-b97e-3e5f70878a10"
-					(reference "J4")
-					(unit 1)
-				)
 			)
 		)
@@
 					(unit 1)
 				)
-			)
-		)
-	)
-	(symbol
-		(lib_id "power:GND")
-		(at 191.77 38.1 0)
-		(mirror y)
-		(unit 1)
-		(exclude_from_sim no)
-		(in_bom yes)
-		(on_board yes)
-		(dnp no)
-		(fields_autoplaced yes)
-		(property "Reference" "#PWR015"
-			(at 191.77 44.45 0)
-			(effects
-				(font
-					(size 1.27 1.27)
-				)
-				(hide yes)
-			)
-		)
-		(property "Value" "GND"
-			(at 191.77 43.18 0)
-			(effects
-				(font
-					(size 1.27 1.27)
-				)
-			)
-		)
-		(property "Footprint" ""
-			(at 191.77 38.1 0)
-			(effects
-				(font
-					(size 1.27 1.27)
-				)
-				(hide yes)
-			)
-		)
-		(property "Datasheet" ""
-			(at 191.77 38.1 0)
-			(effects
-				(font
-					(size 1.27 1.27)
-				)
-				(hide yes)
-			)
-		)
-		(property "Description" "Power symbol creates a global label with name \"GND\" , ground"
-			(at 191.77 38.1 0)
-			(effects
-				(font
-					(size 1.27 1.27)
-				)
-				(hide yes)
-			)
-		)
-		(pin "1"
-		)
-		(instances
-			(project "pylons_boosh_remote_reciver"
-				(path "/f3653ac0-a28a-4ee8-bcf5-236139001455/d08cb7b6-6190-46a9-b97e-3e5f70878a10"
-					(reference "#PWR015")
-					(unit 1)
-				)

Commit message: Add expansion buttons/lamps schematic sheet; schematic cleanup and annotations
- New EXPANSION_BUTTONS_LAMPS.kicad_sch sheet wired into top-level schematic
- Add AB_800T-QT24 symbol library
- ESP32_MCU: wire previously unconnected GPIO pins to BUTTON0-4 and BUTTON_LAMP_PWM_OUT0-4 global labels; add expansion IO bounding box annotation
- POWER: add GND ganging fabrication notes, DCDC USB wiring note, fuse value updated to "10A MINI AUTO BLADE"; routing cleanup
- CONNECTORS: routing and junction cleanup
- BOOSH_TRIGGER: remove stale "1R" errata note
- IDEA.md: add sandbox notes and open questions

Co-Authored-By: Claude Sonnet 4.6 <noreply@anthropic.com>
Connections:
- net GND: no longer J3.2 (Pin_2)
Changed lines of the file:
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@@
 	(paper "A4")
-	(junction
-		(at 132.08 46.99)
-		(diameter 0)
-		(color 0 0 0 0)
-	)
 	(junction
 		(at 55.88 116.84)
@@
 	)
 	(junction
-		(at 134.62 44.45)
-		(diameter 0)
-		(color 0 0 0 0)
-	)
-	(junction
 		(at 53.34 114.3)
 		(diameter 0)
@@
 	)
 	(junction
-		(at 132.08 67.31)
+		(at 138.43 44.45)
 		(diameter 0)
 		(color 0 0 0 0)
@@
 	(wire
 		(pts
-			(xy 132.08 46.99) (xy 134.62 46.99)
-		)
-		(stroke
-			(width 0.508)
-			(type default)
-		)
-	)
-	(wire
-		(pts
 			(xy 100.33 114.3) (xy 130.81 114.3)
 		)
@@
 	(wire
 		(pts
-			(xy 138.43 44.45) (xy 134.62 44.45)
-		)
-		(stroke
-			(width 0.508)
-			(type default)
-		)
-	)
-	(wire
-		(pts
 			(xy 279.4 64.77) (xy 248.92 64.77)
 		)
@@
 	(wire
 		(pts
-			(xy 97.79 67.31) (xy 132.08 67.31)
-		)
-		(stroke
-			(width 0.508)
-			(type default)
-		)
-	)
-	(wire
-		(pts
 			(xy 142.24 67.31) (xy 142.24 69.85)
 		)
@@
 	(wire
 		(pts
+			(xy 138.43 44.45) (xy 138.43 40.64)
+		)
+		(stroke
+			(width 0.508)
+			(type default)
+		)
+	)
+	(wire
+		(pts
 			(xy 100.33 129.54) (xy 100.33 116.84)
 		)
@@
 	(wire
 		(pts
-			(xy 134.62 40.64) (xy 134.62 44.45)
-		)
-		(stroke
-			(width 0.508)
-			(type default)
-		)
-	)
-	(wire
-		(pts
 			(xy 130.81 129.54) (xy 100.33 129.54)
 		)
@@
 	(wire
 		(pts
-			(xy 134.62 46.99) (xy 134.62 49.53)
-		)
-		(stroke
-			(width 0.508)
-			(type default)
-		)
-	)
-	(wire
-		(pts
 			(xy 53.34 114.3) (xy 53.34 121.92)
 		)
@@
 	(wire
 		(pts
+			(xy 130.81 44.45) (xy 138.43 44.45)
+		)
+		(stroke
+			(width 0.508)
+			(type default)
+		)
+	)
+	(wire
+		(pts
 			(xy 274.32 62.23) (xy 248.92 62.23)
 		)
@@
 	(wire
 		(pts
-			(xy 132.08 67.31) (xy 142.24 67.31)
+			(xy 97.79 67.31) (xy 142.24 67.31)
 		)
 		(stroke
@@
 	(wire
 		(pts
-			(xy 130.81 46.99) (xy 132.08 46.99)
-		)
-		(stroke
-			(width 0.508)
-			(type default)
-		)
-	)
-	(wire
-		(pts
 			(xy 142.24 64.77) (xy 205.74 64.77)
 		)
@@
 	(wire
 		(pts
-			(xy 134.62 44.45) (xy 130.81 44.45)
-		)
-		(stroke
-			(width 0.508)
-			(type default)
-		)
-	)
-	(wire
-		(pts
 			(xy 275.59 59.69) (xy 275.59 92.71)
 		)
@@
 		(stroke
 			(width 0)
-			(type default)
-		)
-	)
-	(wire
-		(pts
-			(xy 132.08 46.99) (xy 132.08 67.31)
-		)
-		(stroke
-			(width 0.508)
 			(type default)
 		)
@@
 	(symbol
 		(lib_id "power:+12V")
-		(at 134.62 40.64 0)
+		(at 138.43 40.64 0)
 		(unit 1)
 		(exclude_from_sim no)
@@
 		(dnp no)
 		(property "Reference" "#PWR06"
-			(at 134.62 44.45 0)
+			(at 138.43 44.45 0)
 			(effects
 				(font
@@
 		)
 		(property "Value" "+12V"
-			(at 134.62 35.56 0)
+			(at 138.43 35.56 0)
 			(effects
 				(font
@@
 		)
 		(property "Footprint" ""
-			(at 134.62 40.64 0)
+			(at 138.43 40.64 0)
 			(effects
 				(font
@@
 		)
 		(property "Datasheet" ""
-			(at 134.62 40.64 0)
+			(at 138.43 40.64 0)
 			(effects
 				(font
@@
 		)
 		(property "Description" "Power symbol creates a global label with name \"+12V\""
-			(at 134.62 40.64 0)
+			(at 138.43 40.64 0)
 			(effects
 				(font
@@
 					(unit 1)
 				)
-			)
-		)
-	)
-	(symbol
-		(lib_id "power:GND")
-		(at 134.62 49.53 0)
-		(unit 1)
-		(exclude_from_sim no)
-		(in_bom yes)
-		(on_board yes)
-		(dnp no)
-		(fields_autoplaced yes)
-		(property "Reference" "#PWR014"
-			(at 134.62 55.88 0)
-			(effects
-				(font
-					(size 1.27 1.27)
-				)
-				(hide yes)
-			)
-		)
-		(property "Value" "GND"
-			(at 134.62 54.61 0)
-			(effects
-				(font
-					(size 1.27 1.27)
-				)
-			)
-		)
-		(property "Footprint" ""
-			(at 134.62 49.53 0)
-			(effects
-				(font
-					(size 1.27 1.27)
-				)
-				(hide yes)
-			)
-		)
-		(property "Datasheet" ""
-			(at 134.62 49.53 0)
-			(effects
-				(font
-					(size 1.27 1.27)
-				)
-				(hide yes)
-			)
-		)
-		(property "Description" "Power symbol creates a global label with name \"GND\" , ground"
-			(at 134.62 49.53 0)
-			(effects
-				(font
-					(size 1.27 1.27)
-				)
-				(hide yes)
-			)
-		)
-		(pin "1"
-		)
-		(instances
-			(project "pylons_boosh_remote_reciver"
-				(path "/f3653ac0-a28a-4ee8-bcf5-236139001455/d08cb7b6-6190-46a9-b97e-3e5f70878a10"
-					(reference "#PWR014")
-					(unit 1)
-				)
