File: schematic_electrical/CONNECTORS.kicad_sch (KiCad schematic)
At the start: 9 parts, among them J1 Conn_01x02, J12 Conn_01x03, J15 Conn_01x02, J16 Conn_01x03, J2 Conn_01x02, J3 2-pin red PCB mount connector, J5 2-pin red PCB mount connector

Commit message: Schematic for bar: use ULN2308 for button 12V lamps
Other:
- note added: "NOT POPULATED ON BAR PYLON AS NO LOCAL TANK FOR THERMO AND USING LINE POWER NOT BATTERY"
Changed lines of the file:
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@@
+	)
+	(rectangle
+		(start 12.7 90.17)
+		(end 176.53 154.94)
+		(stroke
+			(width 0)
+			(type dash)
+		)
+		(fill
+			(type none)
+		)
 	)
 	(rectangle
@@
 			)
 		)
+	)
+	(text "NOT POPULATED ON BAR PYLON\nAS NO LOCAL TANK FOR THERMO\nAND USING LINE POWER NOT BATTERY"
+		(exclude_from_sim no)
+		(at 90.678 151.384 0)
+		(effects
+			(font
+				(size 1.27 1.27)
+			)
+		)
